Commit message: 修改urdf

File: assets/r2_v2_with_shell_no_hand/r2v2_with_shell.urdf (robot description, URDF)
Before this commit: robot R2V2, 34 links, 33 joints
Joints:
- joint left_hand_pitch_joint: limit lower=-1.97222205475359 upper=1.97222205475359 effort=36 velocity=9.32005820564972 -> (none); type revolute -> fixed
- joint left_hand_roll_joint: limit lower=-1.0471975511966 upper=1.0471975511966 effort=36 velocity=9.32005820564972 -> (none); type revolute -> fixed
- joint left_hip_roll_joint: limit lower=-0.22689280276 upper=2.44346095279206 effort=130 velocity=14.6607657167524 -> lower=-0.785398163397448 upper=0.785398163397448 effort=130 velocity=14.6607657167524
- joint left_knee_joint: limit lower=-0.530580092606276 upper=2.50629280586386 effort=150 velocity=14.6607657167524 -> lower=0 upper=2.0943951023932 effort=150 velocity=14.6607657167524
- joint right_hand_pitch_joint: limit lower=-1.0471975511966 upper=1.0471975511966 effort=36 velocity=9.32005820564972 -> (none); type revolute -> fixed
- joint right_hand_roll_joint: limit lower=-1.0471975511966 upper=1.0471975511966 effort=36 velocity=9.32005820564972 -> (none); type revolute -> fixed
- joint right_hip_roll_joint: limit lower=-2.44346095279206 upper=0.22689280276 effort=130 velocity=14.6607657167524 -> lower=-0.785398163397448 upper=0.785398163397448 effort=130 velocity=14.6607657167524
- joint right_knee_joint: limit lower=-0.530580092606276 upper=2.50629280586386 effort=150 velocity=14.6607657167524 -> lower=0 upper=2.0943951023932 effort=150 velocity=14.6607657167524
